File: Phase B/PCD_Designs/Uno_Shield_ThermoPro_V2/Uno_Shield_ThermoPro.kicad_pcb (KiCad board)
At the start: 2 copper layers, 68.6 x 53.3 mm, 20 parts, among them J1 Power, J2 Digital/PWM, J3 Analog, J4 Digital/PWM, J5 CONN_GYRO, J6 CONN_DISPLAY, J7 Conn_Temp, SW1 SW_SPST, SW2 SW_SPST, SW3 SW_SPST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

Commit message: final
Parts:
- added G***: LOGO, LOGO, F.Cu at (115.5, 84.5)
- moved R4 0.50 mm to (150.6, 53.5)
Routing:
- net /temp_digital: track 12.9 -> 16.2 mm
- net /button_lock: track 31.0 -> 32.4 mm
- net /button_onoff: track 19.7 -> 20.7 mm
- net /button_units: track 43.0 -> 43.8 mm
- net +5V: track 198.3 -> 198.8 mm
Other:
- board text added: "10"
- board text added: "2"
- board text added: "3"
- board text added: "4"
- board text added: "5"
- board text added: "6"
- board text added: "9"
- board text added: "Analogue Sensor"
- board text added: "MPU6050"
- board text added: "OLED"
- board text added: "R. Lock"
- board text added: "Temp Sensor"
- board text added: "V1 Temp Probe Feb 3 2025 Winston Har"
- board text removed: "Lock"
