File: Phase B/PCD_Designs/Uno_Shield_ThermoPro_V2/Uno_Shield_ThermoPro.kicad_sch (KiCad schematic)
At the start: 20 parts, among them J1 Power, J2 Digital/PWM, J3 Analog, J4 Digital/PWM, J5 CONN_GYRO, J6 CONN_DISPLAY, J7 Conn_Temp, SW1 SW_SPST, SW2 SW_SPST, SW3 SW_SPST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

Commit message: Updated files in V2 folder, new pdf docs and gerber files
Other:
- company: Goncalo Martins -> Winston Har
- title: Uno Shield ThermoPro -> Uno Shield ThermoPro V2
Changed lines of the file:
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@@
 	(paper "A4")
 	(title_block
-		(title "Uno Shield ThermoPro")
-		(date "2025-01-27")
-		(rev "1.0")
-		(company "Goncalo Martins")
+		(title "Uno Shield ThermoPro V2")
+		(date "2025-02-02")
+		(rev "2.0")
+		(company "Winston Har")
 	)
 	(junction

Commit message: schematic edits
Other:
- title: Uno Shield ThermoPro V2 -> Uno Shield ThermoPro V1
Changed lines of the file:
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@@
 	(paper "A4")
 	(title_block
-		(title "Uno Shield ThermoPro V2")
-		(date "2025-02-02")
-		(rev "2.0")
+		(title "Uno Shield ThermoPro V1")
+		(date "2025-02-03")
+		(rev "1.0")
 		(company "Winston Har")
 	)
